File: hardware/V2/diyBMS_CurrentVoltage_ADS1115.kicad_pcb (KiCad board)
At the start: 2 copper layers, 62.2 x 95.6 mm, 53 parts, among them J2 Debug/UPDI, J3 Screw_Terminal_01x04, J4 9x9 PIN connector, J5 9x9 PIN connector, J6 Screw_Terminal_01x02, J7 Screw_Terminal_01x02, J8 PA3/PA4, U1 ACPL-C870, U2 ADS1115IDGS, U3 ACS758xCB-200B-PFF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

Commit message: Added hardware V1, added trimmer to hardware V2, fixed parity between schematic & gerber
Parts:
- removed R18, R19: 10k, Resistor_SMD:R_0805_2012Metric
- added RV1: 10k 10turn, Potentiometer_THT:Potentiometer_Bourns_3299W_Vertical, F.Cu at (56.4, 55.6)
- moved C17 2.82 mm to (59.2, 59.7)
Routing:
- net Net-(U2-AIN3): track 9.07 -> 7.37 mm
- net GND: vias 23 -> 22
